File: cpu3.5e2.brd (EAGLE design)
At the start: 99.7 x 69.8 mm, 111 parts, among them J1 H8WA6A10232, U1 ESP32DEVKITCV4-S, U2 SAMD21MINI, U3 B0505S-1W, U4 B0515S-1W, U5 TFT3-5, U7 POW_E2, X1 DS1002-01-1X19V13, X2 DS1002-01-1X19V13, X3 FH12-20S-1SH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

Commit message: Update cpu3.5e2.brd
Parts:
- moved VD6 0.32 mm to (44.1, 13.3)
- moved VD7 0.32 mm to (44.1, 18.1)
- moved VD8 0.32 mm to (44.1, 8.57)
- moved J3 0.32 mm to (-32.4, -14.6)
Routing:
- net GND: track 117.7 -> 103.8 mm, vias 52 -> 54
- net -VO: track 52.6 -> 55.1 mm
- net V_MOSI: track 203.8 -> 205.2 mm
- net +VO: track 19.4 -> 20.6 mm, vias 2 -> 1
- net V_CLK: track 205.1 -> 206.2 mm
- net V_MISO: track 183.2 -> 184.2 mm
- net +3.3: track 74.4 -> 73.5 mm
- net /OUT: track 98.3 -> 99.0 mm

Commit message: sch
Routing:
- net GND: track 103.8 -> 101.3 mm
Changed lines of the file:
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@@
 <setting verticaltext="down"/>
 </settings>
-<grid distance="6.25" unitdist="mil" unit="mil" style="lines" multiple="1" display="yes" altdistance="0.025" altunitdist="inch" altunit="inch"/>
+<grid distance="6.25" unitdist="mil" unit="mm" style="lines" multiple="1" display="yes" altdistance="0.025" altunitdist="inch" altunit="inch"/>
 <layers>
 <layer number="1" name="Top" color="4" fill="1" visible="yes" active="yes"/>
@@
 <via x="-37.1475" y="1.5875" extent="1-16" drill="0.508"/>
 <via x="-33.9725" y="1.5875" extent="1-16" drill="0.508"/>
-<wire x1="-5.715" y1="22.5425" x2="-8.255" y2="22.5425" width="0.4064" layer="1"/>
 <via x="-34.925" y="24.4475" extent="1-16" drill="0.508"/>
 <contactref element="X8" pad="2"/>
@@
 <wire x1="4.72398125" y1="2.81898125" x2="3.4925" y2="1.5875" width="0.6096" layer="16"/>
 <via x="-12.3825" y="1.5875" extent="1-16" drill="0.508"/>
-<wire x1="-2.055" y1="20.88" x2="-2.0075" y2="20.97056875" width="0" layer="19" extent="16-16"/>
 <wire x1="-42.2275" y1="1.5875" x2="-39.6875" y2="1.5875" width="0.4064" layer="1"/>
 <via x="-19.20875" y="16.03375" extent="1-16" drill="0.508"/>
 <via x="-23.1775" y="16.1925" extent="1-16" drill="0.508"/>
+<wire x1="-2.0075" y1="20.97056875" x2="-2.037953125" y2="20.897046875" width="0.4064" layer="16" curve="-44.998782"/>
+<wire x1="-2.037953125" y1="20.897046875" x2="-2.055" y2="20.88" width="0.4064" layer="16"/>
 </signal>
 <signal name="+3.3V">
@@
 <contactref element="X9" pad="1"/>
 <contactref element="X2" pad="17"/>
-<wire x1="-13.97" y1="28.2575" x2="34.1584875" y2="28.2575" width="0.4064" layer="16"/>
+<wire x1="-13.6525" y1="28.2575" x2="34.1584875" y2="28.2575" width="0.4064" layer="16"/>
 <wire x1="42.9940125" y1="20.955" x2="45.19395" y2="20.955" width="0.4064" layer="16"/>
 <wire x1="46.99" y1="19.15895" x2="46.99" y2="8.46355" width="0.4064" layer="16"/>
@@
 <wire x1="-16.8275" y1="16.6415125" x2="-16.51" y2="15.875" width="0.4064" layer="1" curve="45"/>
 <wire x1="34.1584875" y1="28.2575" x2="36.5125" y2="26.9875" width="0.4064" layer="16" curve="-45"/>
-<wire x1="-13.97" y1="28.2575" x2="-15.0540125" y2="27.8084875" width="0.4064" layer="16" curve="45"/>
-<wire x1="-16.51" y1="25.7175" x2="-16.0609875" y2="26.8015125" width="0.4064" layer="16" curve="-45"/>
-<wire x1="-16.0609875" y1="26.8015125" x2="-15.0540125" y2="27.8084875" width="0.4064" layer="16"/>
+<wire x1="-13.6525" y1="28.2575" x2="-14.19450625" y2="28.03299375" width="0.4064" layer="16" curve="45"/>
+<wire x1="-14.19450625" y1="28.03299375" x2="-16.51" y2="25.7175" width="0.4064" layer="16"/>
 </signal>
 <signal name="BAT-">
@@
 <wire x1="37.7825" y1="24.710525" x2="37.7825" y2="27.94" width="0.4064" layer="1"/>
 <via x="37.7825" y="27.94" extent="1-16" drill="0.5"/>
-<wire x1="35.476965625" y1="29.21" x2="-18.6009875" y2="29.21" width="0.4064" layer="16"/>
+<wire x1="35.476965625" y1="29.21" x2="-17.62125" y2="29.21" width="0.4064" layer="16"/>
 <wire x1="-46.19625" y1="14.2875" x2="-20.79625" y2="14.2875" width="0.4064" layer="16"/>
 <via x="-20.79625" y="14.2875" extent="1-16" drill="0.5"/>
@@
 <wire x1="35.476965625" y1="29.21" x2="37.244734375" y2="28.477765625" width="0.4064" layer="16" curve="-45.000051"/>
 <wire x1="37.244734375" y1="28.477765625" x2="37.7825" y2="27.94" width="0.4064" layer="16"/>
-<wire x1="-18.6009875" y1="29.21" x2="-19.3675" y2="28.8925" width="0.4064" layer="16" curve="45"/>
-<wire x1="-20.0025" y1="27.6225" x2="-19.5534875" y2="28.7065125" width="0.4064" layer="16" curve="-45"/>
-<wire x1="-19.5534875" y1="28.7065125" x2="-19.3675" y2="28.8925" width="0.4064" layer="16"/>
+<wire x1="-17.62125" y1="29.21" x2="-18.976265625" y2="28.648734375" width="0.4064" layer="16" curve="45"/>
+<wire x1="-18.976265625" y1="28.648734375" x2="-20.0025" y2="27.6225" width="0.4064" layer="16"/>
 </signal>
 <signal name="V_MOSI">
@@
 <contactref element="X9" pad="2"/>
 <contactref element="X2" pad="18"/>
-<wire x1="36.111965625" y1="30.1625" x2="-20.32" y2="30.1625" width="0.4064" layer="16"/>
+<wire x1="36.111965625" y1="30.1625" x2="-19.05" y2="30.1625" width="0.4064" layer="16"/>
 <wire x1="-46.19625" y1="11.7475" x2="-29.5275" y2="11.7475" width="0.4064" layer="16"/>
 <via x="-21.9075" y="11.7475" extent="1-16" drill="0.5"/>
@@
 <wire x1="36.111965625" y1="30.1625" x2="37.879734375" y2="29.430265625" width="0.4064" layer="16" curve="-45.000051"/>
 <wire x1="37.879734375" y1="29.430265625" x2="38.998025" y2="28.311975" width="0.4064" layer="16"/>
-<wire x1="-20.32" y1="30.1625" x2="-20.86200625" y2="29.93799375" width="0.4064" layer="16" curve="45"/>
-<wire x1="-20.86200625" y1="29.93799375" x2="-21.2725" y2="29.5275" width="0.4064" layer="16"/>
 <wire x1="-21.9075" y1="27.94" x2="-21.9075" y2="27.994475" width="0.4064" layer="16"/>
-<wire x1="-21.9075" y1="27.994475" x2="-21.2725" y2="29.5275" width="0.4064" layer="16" curve="-45"/>
+<wire x1="-19.05" y1="30.1625" x2="-20.1340125" y2="29.7134875" width="0.4064" layer="16" curve="45"/>
+<wire x1="-20.1340125" y1="29.7134875" x2="-21.9075" y2="27.94" width="0.4064" layer="16"/>
 </signal>
 <signal name="V_CLK">

Commit message: sch
Parts:
- VD3, VD4: device diode-1:DO214AC -> diode:DO214AC
Changed lines of the file:
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@@
 <grid distance="6.25" unitdist="mil" unit="mm" style="lines" multiple="1" display="yes" altdistance="0.025" altunitdist="inch" altunit="inch"/>
 <layers>
-<layer number="1" name="Top" color="4" fill="1" visible="yes" active="yes"/>
+<layer number="1" name="Top" color="4" fill="1" visible="no" active="yes"/>
 <layer number="2" name="Route2" color="1" fill="3" visible="no" active="no"/>
 <layer number="3" name="Route3" color="4" fill="3" visible="no" active="no"/>
@@
 <layer number="28" name="bValues" color="7" fill="1" visible="no" active="yes"/>
 <layer number="29" name="tStop" color="7" fill="3" visible="no" active="yes"/>
-<layer number="30" name="bStop" color="7" fill="6" visible="no" active="yes"/>
+<layer number="30" name="bStop" color="7" fill="6" visible="yes" active="yes"/>
 <layer number="31" name="tCream" color="7" fill="4" visible="no" active="yes"/>
 <layer number="32" name="bCream" color="7" fill="5" visible="no" active="yes"/>
@@
 <layer number="50" name="dxf" color="7" fill="1" visible="no" active="no"/>
 <layer number="51" name="tDocu" color="7" fill="1" visible="no" active="yes"/>
-<layer number="52" name="bDocu" color="7" fill="1" visible="yes" active="yes"/>
+<layer number="52" name="bDocu" color="7" fill="1" visible="no" active="yes"/>
 <layer number="53" name="tGND_GNDA" color="7" fill="1" visible="no" active="no"/>
 <layer number="54" name="bGND_GNDA" color="7" fill="1" visible="no" active="no"/>
@@
 <layer number="220" name="220bmp" color="7" fill="1" visible="no" active="yes"/>
 <layer number="221" name="221bmp" color="7" fill="1" visible="no" active="yes"/>
+<layer number="222" name="222bmp" color="7" fill="1" visible="no" active="yes"/>
 <layer number="223" name="223bmp" color="7" fill="1" visible="no" active="yes"/>
 <layer number="224" name="224bmp" color="7" fill="1" visible="no" active="yes"/>
@@
 </class>
 </classes>
-<designrules name="default *">
+<designrules name="MKlon_E">
 <description language="de">&lt;b&gt;EAGLE Design Rules&lt;/b&gt;
 &lt;p&gt;
@@
 <attribute name="VALUE" x="-5.715" y="-3.4925" size="0.8128" layer="28" font="vector" ratio="10" rot="MR270" align="center"/>
 </element>
-<element name="VD3" library="diode-1" package="DO214AC" value="M4" x="-6.985" y="16.1925" smashed="yes" rot="MR90">
-<attribute name="NAME" x="-5.23875" y="18.25625" size="1.016" layer="26" font="vector" ratio="11" rot="MR90" align="bottom-center"/>
-<attribute name="VALUE" x="-6.985" y="16.8275" size="0.8128" layer="28" font="vector" ratio="10" rot="MR90" align="center"/>
-</element>
-<element name="VD4" library="diode-1" package="DO214AC" value="M4" x="0.635" y="16.1925" smashed="yes" rot="MR90">
-<attribute name="NAME" x="3.4925" y="16.8275" size="1.016" layer="26" font="vector" ratio="11" rot="MR0" align="bottom-center"/>
-<attribute name="VALUE" x="0.635" y="16.8275" size="0.8128" layer="28" font="vector" ratio="10" rot="MR90" align="center"/>
-</element>
 <element name="F1" library="fuse_moro" package="MF-SMDF050" value="MF-SMDF200" x="-6.35" y="-18.415" smashed="yes" rot="MR180">
 <attribute name="NAME" x="-5.715" y="-15.24" size="1.016" layer="26" font="vector" ratio="11" rot="MR0" align="bottom-center"/>
@@
 <attribute name="NAME" x="4.7625" y="-8.255" size="1.016" layer="26" font="vector" ratio="11" rot="MR180" align="bottom-center"/>
 <attribute name="VALUE" x="6.985" y="-9.525" size="1.27" layer="28" rot="MR0"/>
+</element>
+<element name="VD4" library="diode" package="DO214AC" value="M4" x="0.635" y="16.1925" smashed="yes" rot="MR90">
+<attribute name="NAME" x="1.921" y="13.5525" size="1.016" layer="26" font="vector" ratio="11" rot="MR90" align="bottom-center"/>
+<attribute name="VALUE" x="-1.921" y="13.5525" size="1.27" layer="28" ratio="10" rot="MR90"/>
+</element>
+<element name="VD3" library="diode" package="DO214AC" value="M4" x="-6.985" y="16.1925" smashed="yes" rot="MR90">
+<attribute name="NAME" x="-5.699" y="16.0925" size="1.016" layer="26" font="vector" ratio="11" rot="MR90" align="bottom-center"/>
+<attribute name="VALUE" x="-9.541" y="13.5525" size="1.27" layer="28" ratio="10" rot="MR90"/>
 </element>
 </elements>
@@
 <signal name="+18V">
 <contactref element="R6" pad="2"/>
-<contactref element="VD3" pad="A"/>
 <wire x1="-7.13" y1="18.0975" x2="-6.985" y2="18.2425" width="0.4064" layer="16"/>
 <wire x1="-8.626975" y1="17.725525" x2="-9.153025" y2="17.199475" width="0.4064" layer="16"/>
@@
 <wire x1="-5.526975" y1="20.88" x2="-5.9759875" y2="20.6940125" width="0.4064" layer="16" curve="45"/>
 <wire x1="-9.525" y1="12.9690625" x2="-10.1625" y2="12.065" width="0.4064" layer="16" curve="-45"/>
+<contactref element="VD3" pad="A"/>
 </signal>
 <signal name="POW_CH">
@@
 </signal>
 <signal name="BAT+">
-<contactref element="VD4" pad="A"/>
 <contactref element="X3" pad="6"/>
 <wire x1="-0.055" y1="20.88" x2="-0.055" y2="19.90830625" width="0.4064" layer="16"/>
 <wire x1="-0.055" y1="19.90830625" x2="0.635" y2="18.2425" width="0.4064" layer="16" curve="45"/>
+<contactref element="VD4" pad="A"/>
 </signal>
 <signal name="N$61">
@@
 <contactref element="R9" pad="1"/>
 <contactref element="C8" pad="1"/>
-<contactref element="VD4" pad="C"/>
-<contactref element="VD3" pad="C"/>
 <wire x1="-6.985" y1="14.1425" x2="-6.985" y2="14.2875" width="0.4064" layer="16"/>
 <wire x1="-6.985" y1="14.2875" x2="-4.7625" y2="14.2875" width="0.4064" layer="16"/>
@@
 <wire x1="1.905" y1="11.836965625" x2="1.172765625" y2="13.604734375" width="0.4064" layer="16" curve="45.000051"/>
 <wire x1="1.172765625" y1="13.604734375" x2="0.635" y2="14.1425" width="0.4064" layer="16"/>
+<contactref element="VD4" pad="C"/>
+<contactref element="VD3" pad="C"/>
 </signal>
 <signal name="LED_R">
