File: cpu3.5e2.sch (EAGLE design)
At the start: 111 parts, among them J1 H8WA6A10232, J2 0R-JUMPB, J3 0R-JUMPB, U1 ESP32DEVKITCV4-S, U2 SAMD21MINI, U3 B0505S-1W, U4 B0515S-1W, U5 TFT3-5, U7 POW_E2, X1 DS1002-01-1X19V13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

Commit message: sch
Changed lines of the file:
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@@
 <part name="U$28" library="supply" deviceset="AGND" device=""/>
 <part name="U$29" library="microbuilder" deviceset="GND" device="" value=" "/>
-<part name="U$30" library="supply" deviceset="AGND" device=""/>
 <part name="R8" library="rcl_moro" deviceset="R-EU_" device="R0805" value="4k7"/>
 <part name="R25" library="rcl_moro" deviceset="R-EU_" device="R0805" value="4k7"/>
@@
 <instance part="VD11" gate="G$1" x="38.1" y="24.13" smashed="yes" rot="R90">
 <attribute name="NAME" x="40.64" y="25.4" size="1.778" layer="95"/>
-<attribute name="VALUE" x="40.64" y="20.32" size="1.778" layer="96"/>
+<attribute name="VALUE" x="40.64" y="22.86" size="1.778" layer="96"/>
 </instance>
 <instance part="VD12" gate="G$1" x="48.26" y="24.13" smashed="yes" rot="R270">
 <attribute name="NAME" x="50.8" y="25.4" size="1.778" layer="95"/>
-<attribute name="VALUE" x="40.64" y="20.32" size="1.778" layer="96"/>
+<attribute name="VALUE" x="40.64" y="22.86" size="1.778" layer="96"/>
 </instance>
 <instance part="U3" gate="G$1" x="175.26" y="144.78" smashed="yes">
@@
 </instance>
 <instance part="U$51" gate="G$1" x="154.94" y="134.62" rot="MR0"/>
-<instance part="GND" gate="G$1" x="10.16" y="20.32" smashed="yes" rot="R270">
-<attribute name="VALUE" x="7.62" y="22.86" size="1.778" layer="96"/>
+<instance part="GND" gate="G$1" x="10.16" y="22.86" smashed="yes" rot="R270">
+<attribute name="VALUE" x="7.62" y="25.4" size="1.778" layer="96"/>
 </instance>
 <instance part="C13" gate="G$1" x="203.2" y="144.78" smashed="yes">
@@
 <attribute name="VALUE" x="208.28" y="132.08" size="1.778" layer="95" rot="R180"/>
 </instance>
-<instance part="AGND" gate="G$1" x="30.48" y="20.32" smashed="yes" rot="R270">
-<attribute name="VALUE" x="27.94" y="22.86" size="1.778" layer="96"/>
+<instance part="AGND" gate="G$1" x="30.48" y="22.86" smashed="yes" rot="R270">
+<attribute name="VALUE" x="27.94" y="25.4" size="1.778" layer="96"/>
 </instance>
 <instance part="R18" gate="G$1" x="48.26" y="86.36" smashed="yes">
@@
 <instance part="U$28" gate="VR1" x="220.98" y="55.88" smashed="yes"/>
 <instance part="U$29" gate="G$1" x="210.82" y="55.88"/>
-<instance part="U$30" gate="VR1" x="43.18" y="15.24" smashed="yes"/>
 <instance part="R25" gate="G$1" x="215.9" y="116.84" smashed="yes" rot="R90">
 <attribute name="NAME" x="218.44" y="119.38" size="1.778" layer="95"/>
@@
 <pinref part="GND" gate="G$1" pin="P"/>
 <pinref part="U$11" gate="G$1" pin="GND"/>
+<wire x1="10.16" y1="20.32" x2="10.16" y2="17.78" width="0.1524" layer="91"/>
 </segment>
 <segment>
@@
 <pinref part="U$58" gate="VR1" pin="AGND"/>
 <pinref part="AGND" gate="G$1" pin="P"/>
-</segment>
-<segment>
+<wire x1="30.48" y1="20.32" x2="30.48" y2="17.78" width="0.1524" layer="91"/>
 <pinref part="VD12" gate="G$1" pin="C"/>
-<wire x1="48.26" y1="17.78" x2="48.26" y2="21.59" width="0.1524" layer="91"/>
-<wire x1="43.18" y1="17.78" x2="48.26" y2="17.78" width="0.1524" layer="91"/>
-<pinref part="U$30" gate="VR1" pin="AGND"/>
+<wire x1="48.26" y1="20.32" x2="48.26" y2="21.59" width="0.1524" layer="91"/>
 <pinref part="VD11" gate="G$1" pin="A"/>
-<wire x1="38.1" y1="17.78" x2="38.1" y2="21.59" width="0.1524" layer="91"/>
-<wire x1="38.1" y1="17.78" x2="43.18" y2="17.78" width="0.1524" layer="91"/>
-<junction x="43.18" y="17.78"/>
-</segment>
-<segment>
+<wire x1="38.1" y1="20.32" x2="38.1" y2="21.59" width="0.1524" layer="91"/>
+<wire x1="38.1" y1="20.32" x2="48.26" y2="20.32" width="0.1524" layer="91"/>
+<wire x1="30.48" y1="20.32" x2="38.1" y2="20.32" width="0.1524" layer="91"/>
+<junction x="30.48" y="20.32"/>
+<junction x="38.1" y="20.32"/>
+</segment>
+<segment>

Commit message: sch
Parts:
- VD3, VD4: device diode-1:SS16 -> diode:DIODE-DO214AC
Other:
- note added: "MKlon3.5 cpu3.5eX"
- note added: "OlMoro 2024"
- note removed: "MKlon3.5 cpu3.5vX"
- note removed: "OlMoro 2023"
Changed lines of the file:
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@@
 <part name="C11" library="rcl_moro" deviceset="C-EU" device="C0805" value="10n"/>
 <part name="VD5" library="diode-1" deviceset="SS16" device=""/>
-<part name="VD3" library="diode-1" deviceset="SS16" device="" value="M4"/>
-<part name="VD4" library="diode-1" deviceset="SS16" device="" value="M4"/>
 <part name="F1" library="fuse_moro" deviceset="MF-SMDF" device="" technology="200"/>
 <part name="U$55" library="microbuilder" deviceset="GND" device="" value=" "/>
@@
 <part name="R8" library="rcl_moro" deviceset="R-EU_" device="R0805" value="4k7"/>
 <part name="R25" library="rcl_moro" deviceset="R-EU_" device="R0805" value="4k7"/>
+<part name="VD4" library="diode" deviceset="DIODE-" device="DO214AC" value="M4"/>
+<part name="VD3" library="diode" deviceset="DIODE-" device="DO214AC" value="M4"/>
 </parts>
 <sheets>
@@
 <text x="233.68" y="111.76" size="1.778" layer="91">(VSPI_SS)</text>
 <text x="177.8" y="10.16" size="3.048" layer="91">MKlon3.5
-cpu3.5vX</text>
-<text x="226.06" y="20.32" size="2.1844" layer="94" ratio="11">OlMoro 2023</text>
+cpu3.5eX</text>
+<text x="226.06" y="20.32" size="2.1844" layer="94" ratio="11">OlMoro 2024</text>
 <text x="68.58" y="40.64" size="1.778" layer="91">(CS)</text>
 <text x="68.58" y="43.18" size="1.778" layer="91">(RST)</text>
@@
 <plain>
 <text x="177.8" y="10.16" size="3.048" layer="91">MKlon3.5
-cpu3.5vX</text>
+cpu3.5eX</text>
 <text x="142.24" y="78.74" size="1.778" layer="91">PA16 TCC2_CH0 (TCC2/WO[0])</text>
 <text x="124.46" y="121.92" size="1.778" layer="95" rot="R180">(pow 180mA)</text>
-<text x="223.52" y="20.32" size="2.1844" layer="94" ratio="11">OlMoro 2023</text>
+<text x="223.52" y="20.32" size="2.1844" layer="94" ratio="11">OlMoro 2024</text>
 <text x="129.54" y="124.46" size="1.778" layer="91">  R11
 (2k2  7v)
@@
 <attribute name="VALUE" x="86.36" y="132.08" size="1.778" layer="96" rot="R180"/>
 </instance>
-<instance part="VD3" gate="G$1" x="22.86" y="152.4" smashed="yes">
-<attribute name="NAME" x="25.4" y="149.86" size="1.778" layer="95" rot="R180"/>
-<attribute name="VALUE" x="25.4" y="147.32" size="1.778" layer="96" rot="R180"/>
-</instance>
-<instance part="VD4" gate="G$1" x="27.94" y="157.48" smashed="yes" rot="R270">
-<attribute name="NAME" x="25.4" y="162.56" size="1.778" layer="95" rot="R180"/>
-<attribute name="VALUE" x="25.4" y="160.02" size="1.778" layer="96" rot="R180"/>
-</instance>
 <instance part="F1" gate="A" x="132.08" y="152.4" smashed="yes">
 <attribute name="NAME" x="137.16" y="149.733" size="1.778" layer="95" rot="R180"/>
@@
 <attribute name="NAME" x="218.44" y="119.38" size="1.778" layer="95"/>
 <attribute name="VALUE" x="218.44" y="116.84" size="1.778" layer="96"/>
+</instance>
+<instance part="VD4" gate="G$1" x="27.94" y="157.48" smashed="yes" rot="R270">
+<attribute name="NAME" x="20.32" y="157.9626" size="1.778" layer="95"/>
+<attribute name="VALUE" x="22.86" y="160.2486" size="1.778" layer="96"/>
+</instance>
+<instance part="VD3" gate="G$1" x="22.86" y="152.4" smashed="yes">
+<attribute name="NAME" x="25.4" y="149.3774" size="1.778" layer="95" rot="R180"/>
+<attribute name="VALUE" x="25.4" y="147.0914" size="1.778" layer="96" rot="R180"/>
 </instance>
 </instances>
@@
 <net name="+18V" class="0">
 <segment>
-<pinref part="VD3" gate="G$1" pin="A"/>
 <wire x1="20.32" y1="152.4" x2="12.7" y2="152.4" width="0.1524" layer="91"/>
 <label x="20.32" y="154.94" size="1.778" layer="95" rot="R180"/>
+<pinref part="VD3" gate="G$1" pin="A"/>
 </segment>
 <segment>
@@
 <net name="BAT+" class="0">
 <segment>
-<pinref part="VD4" gate="G$1" pin="A"/>
 <label x="30.48" y="162.56" size="1.778" layer="95" rot="R90"/>
 <wire x1="27.94" y1="170.18" x2="27.94" y2="160.02" width="0.1524" layer="91"/>
+<pinref part="VD4" gate="G$1" pin="A"/>
 </segment>
 <segment>
@@
 <pinref part="C8" gate="G$1" pin="1"/>
 <wire x1="43.18" y1="149.86" x2="43.18" y2="152.4" width="0.1524" layer="91"/>
-<pinref part="VD4" gate="G$1" pin="C"/>
 <wire x1="27.94" y1="154.94" x2="27.94" y2="152.4" width="0.1524" layer="91"/>
 <wire x1="27.94" y1="152.4" x2="40.64" y2="152.4" width="0.1524" layer="91"/>
 <junction x="40.64" y="152.4"/>
-<pinref part="VD3" gate="G$1" pin="C"/>
 <wire x1="27.94" y1="152.4" x2="25.4" y2="152.4" width="0.1524" layer="91"/>
 <junction x="27.94" y="152.4"/>
 <label x="35.56" y="154.94" size="1.778" layer="95" rot="R180"/>
-</segment>
-<segment>
+<pinref part="VD4" gate="G$1" pin="C"/>
+<pinref part="VD3" gate="G$1" pin="C"/>
+</segment>
+<segment>
